File: NewPCB/NewPCB.kicad_sch (KiCad schematic)
At the start: 0 parts

Commit message: added PCB work
Parts:
- added J2: B4B-XH-A, CONN_B4B-XH-A_JST, symbol 2025-09-13_16-31-34:B4B-XH-A
- added U1: DEV-15583, DEV-15583:MODULE_DEV-15583, symbol Teensy:DEV-15583
Connections:
- new net: J2.2, U1.18
- new net: J2.3, U1.19
- new net: J2.1, U1.3.3V_2
- new net GND: J2.4, U1.G1, U1.G2, U1.G3
